File: ELEC/Project/SoundHive.sch (KiCad schematic (older format))
At the start: 1 part

Commit message: Getting started
Parts:
- added C?: C, ~, symbol C
- added R?: R, ~, symbol R
- gave numbers to parts that had none: 1
Changed lines of the file:
@@
 LIBS:ClassD_Audio
 LIBS:valves
+LIBS:Zilog
+LIBS:zetex
+LIBS:Xicor
+LIBS:Worldsemi
+LIBS:wiznet
+LIBS:video
+LIBS:ttl_ieee
+LIBS:triac_thyristor
+LIBS:transf
+LIBS:switches
+LIBS:supertex
+LIBS:stm32
+LIBS:stm8
+LIBS:silabs
+LIBS:sensors
+LIBS:RFSolutions
+LIBS:rfcom
+LIBS:relays
+LIBS:references
+LIBS:pspice
+LIBS:Power_Management
+LIBS:powerint
+LIBS:Oscillators
+LIBS:onsemi
+LIBS:nxp_armmcu
+LIBS:nxp
+LIBS:nordicsemi
+LIBS:msp430
+LIBS:motors
+LIBS:motor_drivers
+LIBS:modules
+LIBS:microchip_pic32mcu
+LIBS:microchip_pic24mcu
+LIBS:microchip_pic18mcu
+LIBS:microchip_pic16mcu
+LIBS:microchip_pic12mcu
+LIBS:microchip_pic10mcu
+LIBS:microchip_dspic33dsc
+LIBS:mechanical
+LIBS:maxim
+LIBS:logo
+LIBS:LEM
+LIBS:leds
+LIBS:Lattice
+LIBS:ir
+LIBS:intersil
+LIBS:infineon
+LIBS:hc11
+LIBS:graphic
+LIBS:gennum
+LIBS:ftdi
+LIBS:ESD_Protection
+LIBS:elec-unifil
+LIBS:diode
+LIBS:dc-dc
+LIBS:cmos_ieee
+LIBS:brooktre
+LIBS:bosch
+LIBS:bbd
+LIBS:battery_management
+LIBS:analog_devices
+LIBS:Altera
+LIBS:allegro
+LIBS:actel
+LIBS:ac-dc
+LIBS:74xgxx
 LIBS:SoundHive-cache
 EELAYER 27 0
@@
 $EndDescr
 $Comp
-L TPA3106D1 U?
+L TPA3106D1 U1
 U 1 1 5927C849
 P 5150 3050
-F 0 "U?" H 4250 3800 60  0000 C CNN
+F 0 "U1" H 4250 3800 60  0000 C CNN
 F 1 "TPA3106D1" H 4450 3900 60  0000 C CNN
 F 2 "~" H 4850 3100 60  0000 C CNN
@@
 	1    0    0    -1
 $EndComp
+$Comp
+L R R?
+U 1 1 5927C8A1
+P 2900 3150
+F 0 "R?" V 2980 3150 40  0000 C CNN
+F 1 "R" V 2907 3151 40  0000 C CNN
+F 2 "~" V 2830 3150 30  0000 C CNN
+F 3 "~" H 2900 3150 30  0000 C CNN
+	1    2900 3150
+	1    0    0    -1
+$EndComp
+$Comp
+L C C?
+U 1 1 5927C8BA
+P 3250 4100
+F 0 "C?" H 3250 4200 40  0000 L CNN
+F 1 "C" H 3256 4015 40  0000 L CNN
+F 2 "~" H 3288 3950 30  0000 C CNN
+F 3 "~" H 3250 4100 60  0000 C CNN
+	1    3250 4100
+	1    0    0    -1
+$EndComp
