File: ELEC/40W_Amp/SoundHive.kicad_pcb (KiCad board)
At the start: 2 copper layers, 0 parts

Commit message: Paths updated and stuff
Parts:
- added J1: CONN_01X08, Pin_Headers:Pin_Header_Angled_1x08_Pitch2.54mm, F.Cu at (129.5, 102.9)
- added J2: CONN_01X08, Pin_Headers:Pin_Header_Angled_1x08_Pitch2.54mm, F.Cu at (176.5, 118.1)
- added U1: TPA3106D1, Pin_Headers:Pin_Header_Angled_1x32_Pitch1.27mm, F.Cu at (108.0, 100.3)
Other:
- net class Default: clearance 0.254 -> 0.2; trace_width 0.254 -> 0.25; via_dia 0.889 -> 0.6; via_drill 0.635 -> 0.4
- rule trace_clearance: 0.254 -> 0.2
- rule trace_min: 0.254 -> 0.2
- rule via_min_drill: 0.508 -> 0.3
- rule via_min_size: 0.889 -> 0.4
