File: ELEC/40W_Amp/SoundHive.sch (KiCad schematic (older format))
At the start: 33 parts, among them J1 CONN_01X08, J2 CONN_01X08, J3 Screw_Terminal_1x02, J4 CONN_01X02_MALE, J5 CONN_01X02_MALE, J6 CONN_01X02_MALE, J7 CONN_01X03_MALE, U1 TPA3106D1

Commit message: V1.01, board ordered. June 14th, 2017, OSH Park.
Parts:
- added J8: CONN_01X01, Via:10mil_Via, symbol CONN_01X01
Connections:
- net +24V: now also U1.29 (nSHUTDOWN)
- net GND: now also U1.30 (MUTE), U1.33 (EP)
- net at U1.31 (FAULT): now also J8.1 (P1)
Changed lines of the file:
@@
 Wire Wire Line
 	4150 3100 3600 3100
+$Comp
+L GND #PWR022
+U 1 1 59423AE3
+P 5050 2450
+F 0 "#PWR022" H 5050 2200 50  0001 C CNN
+F 1 "GND" H 5050 2300 50  0000 C CNN
+F 2 "" H 5050 2450 50  0001 C CNN
+F 3 "" H 5050 2450 50  0001 C CNN
+	1    5050 2450
+	1    0    0    -1
+$EndComp
+Wire Wire Line
+	5600 2650 5200 2650
+Wire Wire Line
+	5200 2650 5200 2450
+Wire Wire Line
+	5200 2450 5050 2450
+$Comp
+L GND #PWR023
+U 1 1 59425159
+P 5900 2500
+F 0 "#PWR023" H 5900 2250 50  0001 C CNN
+F 1 "GND" H 5900 2350 50  0000 C CNN
+F 2 "" H 5900 2500 50  0001 C CNN
+F 3 "" H 5900 2500 50  0001 C CNN
+	1    5900 2500
+	-1   0    0    1
+$EndComp
+Wire Wire Line
+	5900 2650 5900 2500
+Connection ~ 6000 1650
+Wire Wire Line
+	6000 1650 6000 2650
+$Comp
+L CONN_01X01 J8
+U 1 1 59428BD9
+P 5800 2450
+F 0 "J8" V 5900 2500 50  0000 C CNN
+F 1 "CONN_01X01" V 5900 2450 50  0001 C CNN
+F 2 "Via:10mil_Via" H 5800 2450 50  0001 C CNN
+F 3 "" H 5800 2450 50  0001 C CNN
+	1    5800 2450
+	0    -1   -1   0
+$EndComp
 $EndSCHEMATC

Commit message: Added CSV
Parts:
- C1, C14, C15, C17, C2, C4, C6, C7, C8, C9: Part Number (none) -> UMK212BJ105KG-T
- C10, C11: Part Number (none) -> UMK212B7224KG-T
- C12, C13: Part Number (none) -> C0805C102J5GACTU
- C16: Part Number (none) -> GRM21BR6YA106KE43L
- R1, R2, R6: Part Number (none) -> RMCF0805JT100K
- R3: Part Number (none) -> RC0805FR-07100KL
- R4, R5: value 20R 1/4 W, 5% -> 20R 1/4 W - 1%; Part Number (none) -> RC0805FR-0720RL
- U1: Part Number (none) -> TPA3106D1
Changed lines of the file:
@@
 F 2 "Houseings_QFP_Walker:LQFP-32_7x7mm_Pitch0.8mm-EP" H 5650 3500 60  0001 C CNN
 F 3 "~" H 5650 3500 60  0000 C CNN
+F 4 "TPA3106D1" H 6000 3500 60  0001 C CNN "Part Number"
 	1    6000 3500
 	1    0    0    -1
@@
 F 2 "Capacitors_SMD:C_0805" H 4338 2950 50  0001 C CNN
 F 3 "" H 4300 3100 50  0001 C CNN
+F 4 "UMK212BJ105KG-T" H 4300 3100 60  0001 C CNN "Part Number"
 	1    4300 3100
 	0    1    1    0
@@
 F 2 "Capacitors_SMD:C_0805" H 4338 3250 50  0001 C CNN
 F 3 "" H 4300 3400 50  0001 C CNN
+F 4 "UMK212BJ105KG-T" H 4300 3400 60  0001 C CNN "Part Number"
 	1    4300 3400
 	0    1    1    0
@@
 F 2 "Capacitors_SMD:C_0805" H 6938 1850 50  0001 C CNN
 F 3 "" H 6900 2000 50  0001 C CNN
+F 4 "UMK212BJ105KG-T" H 6900 2000 60  0001 C CNN "Part Number"
 	1    6900 2000
 	-1   0    0    1
@@
 F 2 "Capacitors_SMD:C_0805" H 6338 5000 50  0001 C CNN
 F 3 "" H 6300 5150 50  0001 C CNN
+F 4 "UMK212BJ105KG-T" H 6300 5150 60  0001 C CNN "Part Number"
 	1    6300 5150
 	-1   0    0    1
@@
 F 2 "Capacitors_SMD:C_0805" H 8488 3150 50  0001 C CNN
 F 3 "" H 8450 3300 50  0001 C CNN
+F 4 "UMK212BJ105KG-T" H 8450 3300 60  0001 C CNN "Part Number"
 	1    8450 3300
 	-1   0    0    1
@@
 F 2 "Capacitors_SMD:C_0805" H 8488 3550 50  0001 C CNN
 F 3 "" H 8450 3700 50  0001 C CNN
+F 4 "UMK212BJ105KG-T" H 8450 3700 60  0001 C CNN "Part Number"
 	1    8450 3700
 	-1   0    0    1
@@
 F 2 "Capacitors_SMD:C_0805" H 7438 2450 50  0001 C CNN
 F 3 "" H 7400 2600 50  0001 C CNN
+F 4 "C0805C102J5GACTU" H 7400 2600 60  0001 C CNN "Part Number"
 	1    7400 2600
 	-1   0    0    1
@@
 P 7400 2050
 F 0 "R4" V 7600 2050 50  0000 C CNN
-F 1 "20R 1/4 W, 5%" V 7500 2050 50  0000 C CNN
+F 1 "20R 1/4 W - 1%" V 7500 2050 50  0000 C CNN
 F 2 "Resistors_SMD:R_1206" V 7330 2050 50  0001 C CNN
 F 3 "" H 7400 2050 50  0001 C CNN
+F 4 "RC0805FR-0720RL" V 7400 2050 60  0001 C CNN "Part Number"
 	1    7400 2050
 	1    0    0    -1
@@
 F 2 "Capacitors_SMD:C_0805" H 7438 4000 50  0001 C CNN
 F 3 "" H 7400 4150 50  0001 C CNN
+F 4 "C0805C102J5GACTU" H 7400 4150 60  0001 C CNN "Part Number"
 	1    7400 4150
 	-1   0    0    1
@@
 F 2 "Capacitors_SMD:C_0805" H 7288 3050 50  0001 C CNN
 F 3 "" H 7250 3200 50  0001 C CNN
+F 4 "UMK212B7224KG-T" H 7250 3200 60  0001 C CNN "Part Number"
 	1    7250 3200
 	-1   0    0    1
@@
 F 2 "Capacitors_SMD:C_0805" H 7288 3650 50  0001 C CNN
 F 3 "" H 7250 3800 50  0001 C CNN
+F 4 "UMK212B7224KG-T" H 7250 3800 60  0001 C CNN "Part Number"
 	1    7250 3800
 	-1   0    0    1
@@
 F 2 "Capacitors_SMD:C_0805" H 5788 5000 50  0001 C CNN
 F 3 "" H 5750 5150 50  0001 C CNN
+F 4 "UMK212BJ105KG-T" H 5750 5150 60  0001 C CNN "Part Number"
 	1    5750 5150
 	-1   0    0    1
@@
 F 2 "Capacitors_SMD:C_0805" H 5488 5000 50  0001 C CNN
 F 3 "" H 5450 5150 50  0001 C CNN
+F 4 "UMK212BJ105KG-T" H 5450 5150 60  0001 C CNN "Part Number"
 	1    5450 5150
 	-1   0    0    1
@@
 F 2 "Capacitors_SMD:C_0805" H 5238 5000 50  0001 C CNN
 F 3 "" H 5200 5150 50  0001 C CNN
+F 4 "UMK212BJ105KG-T" H 5200 5150 60  0001 C CNN "Part Number"
 	1    5200 5150
 	-1   0    0    1
@@
 F 2 "Resistors_SMD:R_0805" V 4880 5150 50  0001 C CNN
 F 3 "" H 4950 5150 50  0001 C CNN
+F 4 "RC0805FR-07100KL" V 4950 5150 60  0001 C CNN "Part Number"
 	1    4950 5150
 	1    0    0    -1
@@
 F 2 "Resistors_SMD:R_0805" V 4230 4450 50  0001 C CNN
 F 3 "" H 4300 4450 50  0001 C CNN
+F 4 "RMCF0805JT100K" V 4300 4450 60  0001 C CNN "Part Number"
 	1    4300 4450
 	1    0    0    -1
@@
 F 2 "Resistors_SMD:R_0805" V 4530 4450 50  0001 C CNN
 F 3 "" H 4600 4450 50  0001 C CNN
+F 4 "RMCF0805JT100K" V 4600 4450 60  0001 C CNN "Part Number"
 	1    4600 4450
 	1    0    0    -1
@@
 P 7400 4700
 F 0 "R5" V 7600 4700 50  0000 C CNN
-F 1 "20R 1/4 W, 5%" V 7500 4700 50  0000 C CNN
+F 1 "20R 1/4 W - 1%" V 7500 4700 50  0000 C CNN
 F 2 "Resistors_SMD:R_1206" V 7330 4700 50  0001 C CNN
 F 3 "" H 7400 4700 50  0001 C CNN
+F 4 "RC0805FR-0720RL" V 7400 4700 60  0001 C CNN "Part Number"
 	1    7400 4700
 	1    0    0    -1
@@
 F 2 "Resistors_SMD:R_0805" V 4880 4050 50  0001 C CNN
 F 3 "" H 4950 4050 50  0001 C CNN
+F 4 "RMCF0805JT100K" V 4950 4050 60  0001 C CNN "Part Number"
 	1    4950 4050
 	1    0    0    -1
@@
 F 2 "Capacitors_SMD:C_0805" H 5588 1900 50  0001 C CNN
 F 3 "" H 5550 2050 50  0001 C CNN
+F 4 "UMK212BJ105KG-T" H 5550 2050 60  0001 C CNN "Part Number"
 	1    5550 2050
 	-1   0    0    1
@@
 F 2 "Capacitors_SMD:C_0805" H 5288 1900 50  0001 C CNN
 F 3 "" H 5250 2050 50  0001 C CNN
+F 4 "GRM21BR6YA106KE43L" H 5250 2050 60  0001 C CNN "Part Number"
 	1    5250 2050
 	-1   0    0    1

Commit message: Traded connector for something that actually fits
Parts:
- J3: footprint Connectors_Terminal_Blocks.pretty:TerminalBlock_Pheonix_MKDS1.5-2pol -> Connectors_Terminal_Blocks.pretty:TerminalBlock_OSTTC022162
Changed lines of the file:
@@
 F 0 "J3" H 9600 3750 50  0000 C TNN
 F 1 "Screw_Terminal_1x02" V 9450 3500 50  0000 C TNN
-F 2 "Connectors_Terminal_Blocks.pretty:TerminalBlock_Pheonix_MKDS1.5-2pol" H 9600 3275 50  0001 C CNN
+F 2 "Connectors_Terminal_Blocks.pretty:TerminalBlock_OSTTC022162" H 9600 3275 50  0001 C CNN
 F 3 "" H 9575 3500 50  0001 C CNN
 F 4 "1715721" H 9600 3500 60  0001 C CNN "Part Number"
